Commit message: Created loop world and adapted car with IMU and steering

File: urdf/racecar.urdf (robot description, URDF)
Before this commit: robot racecar, 10 links, 9 joints
Links:
- added link imu_link, mass 0.01; collision box size=0.02 0.02 0.01; visual box size=0.02 0.02 0.01
Joints:
- added joint imu_joint: type fixed, parent base_link, child imu_link, origin xyz=-0.08 0.0 0.0 rpy=0 0 0
- joint left_steering_hinge_joint: limit lower=-1.0 upper=1.0 effort=10 velocity=100 -> lower=-0.5236 upper=0.5236 effort=10 velocity=100
- joint right_steering_hinge_joint: limit lower=-1.0 upper=1.0 effort=10 velocity=100 -> lower=-0.5236 upper=0.5236 effort=10 velocity=100; type continuous -> revolute
